Commit message: Add initial version of simulation

File: src/open_manipulator_description/urdf/open_manipulator_robot.xacro (robot description, xacro)
@@ -5,5 +5,5 @@
   <link name="world"/>
   <joint name="world_fixed" type="fixed">
-    <origin xyz="0 0 0" rpy="0 0 0"/>
+    <origin xyz="0 0 0.08" rpy="0 0 0"/>
     <parent link="world"/>
     <child link="link1"/>

Commit message: Add robot spawner to simulation bringup

File: src/open_manipulator_description/urdf/open_manipulator_robot.xacro (robot description, xacro)
@@ -5,5 +5,5 @@
   <link name="world"/>
   <joint name="world_fixed" type="fixed">
-    <origin xyz="0 0 0.08" rpy="0 0 0"/>
+    <origin xyz="0 0 0.05" rpy="0 0 0"/>
     <parent link="world"/>
     <child link="link1"/>

Commit message: Add base for manipulator

File: src/open_manipulator_description/urdf/open_manipulator_robot.xacro (robot description, xacro)
@@ -4,7 +4,24 @@
   <xacro:include filename="$(find open_manipulator_description)/urdf/open_manipulator.xacro" />
   <link name="world"/>
+  <link name="base">
+      <visual>
+        <geometry>
+          <cylinder length="0.6" radius="0.2"/>
+        </geometry>
+      </visual>
+      <collision>
+        <geometry>
+          <cylinder length="0.6" radius="0.2"/>
+        </geometry>
+      </collision>
+   </link>
   <joint name="world_fixed" type="fixed">
     <origin xyz="0 0 0.05" rpy="0 0 0"/>
     <parent link="world"/>
+    <child link="base"/>
+  </joint>
+   <joint name="based_fixed" type="fixed">
+    <origin xyz="0 0 0.3" rpy="0 0 0"/>
+    <parent link="base"/>
     <child link="link1"/>
   </joint>

Commit message: Small refactor of urdf files

File: src/open_manipulator_description/urdf/open_manipulator_robot.xacro (robot description, xacro)
@@ -4,24 +4,28 @@
   <xacro:include filename="$(find open_manipulator_description)/urdf/open_manipulator.xacro" />
   <xacro:include filename="$(find open_manipulator_description)/urdf/ros2_control.xacro" />
+  <xacro:property name="base_link_hight" value="0.3"/>
+  <xacro:property name="base_link_radius" value="0.3"/>
+  <xacro:property name="offset_from_ground_to_base_link" value="${base_link_hight/2 + 0.05}"/>
+  <xacro:property name="offset_from_base_link_link1" value="${base_link_hight/2 + 0.01}"/>
   <link name="world"/>
   <link name="base_link">
       <visual>
         <geometry>
-          <cylinder length="0.3" radius="0.3"/>
+          <cylinder length="${base_link_hight}" radius="${base_link_radius}"/>
         </geometry>
       </visual>
       <collision>
         <geometry>
-          <cylinder length="0.3" radius="0.3"/>
+          <cylinder length="${base_link_hight}" radius="${base_link_radius}"/>
         </geometry>
       </collision>
    </link>
   <joint name="world_fixed" type="fixed">
-    <origin xyz="0 0 0.2" rpy="0 0 0"/>
+    <origin xyz="0 0 ${offset_from_ground_to_base_link}" rpy="0 0 0"/>
     <parent link="world"/>
     <child link="base_link"/>
   </joint>
-   <joint name="based_fixed" type="fixed">
-    <origin xyz="0 0 0.16" rpy="0 0 0"/>
+  <joint name="based_fixed" type="fixed">
+    <origin xyz="0 0 ${offset_from_base_link_link1}" rpy="0 0 0"/>
     <parent link="base_link"/>
     <child link="link1"/>
