Commit message: Update path to *.stl files

File: src/open_manipulator_description/urdf/open_manipulator.xacro (robot description, xacro)
@@ -5,12 +5,12 @@
       <origin xyz="0 0 0" rpy="0 0 0"/>
       <geometry>
-        <mesh filename="package://open_manipulator_description/meshes/chain_link1.stl" scale="0.001 0.001 0.001"/>
-      </geometry>
-      <material name="grey"/>
-    </visual>
-    <collision>
-      <origin xyz="0 0 0" rpy="0 0 0"/>
-      <geometry>
-        <mesh filename="package://open_manipulator_description/meshes/chain_link1.stl" scale="0.001 0.001 0.001"/>
+        <mesh filename="file://$(find open_manipulator_description)/meshes/chain_link1.stl" scale="0.001 0.001 0.001"/>
+      </geometry>
+      <material name="grey"/>
+    </visual>
+    <collision>
+      <origin xyz="0 0 0" rpy="0 0 0"/>
+      <geometry>
+        <mesh filename="file://$(find open_manipulator_description)/meshes/chain_link1.stl" scale="0.001 0.001 0.001"/>
       </geometry>
     </collision>
@@ -34,5 +34,5 @@
       <origin xyz="0 0 0.019" rpy="0 0 0"/>
       <geometry>
-        <mesh filename="package://open_manipulator_description/meshes/chain_link2.stl" scale="0.001 0.001 0.001"/>
+        <mesh filename="file://$(find open_manipulator_description)/meshes/chain_link2.stl" scale="0.001 0.001 0.001"/>
       </geometry>
       <material name="grey"/>
@@ -41,5 +41,5 @@
       <origin xyz="0 0 0.019" rpy="0 0 0"/>
       <geometry>
-        <mesh filename="package://open_manipulator_description/meshes/chain_link2.stl" scale="0.001 0.001 0.001"/>
+        <mesh filename="file://$(find open_manipulator_description)/meshes/chain_link2.stl" scale="0.001 0.001 0.001"/>
       </geometry>
     </collision>
@@ -63,12 +63,12 @@
       <origin xyz="0 0 0" rpy="0 0 0"/>
       <geometry>
-        <mesh filename="package://open_manipulator_description/meshes/chain_link3.stl" scale="0.001 0.001 0.001"/>
-      </geometry>
-      <material name="grey"/>
-    </visual>
-    <collision>
-      <origin xyz="0 0 0" rpy="0 0 0"/>
-      <geometry>
-        <mesh filename="package://open_manipulator_description/meshes/chain_link3.stl" scale="0.001 0.001 0.001"/>
+        <mesh filename="file://$(find open_manipulator_description)/meshes/chain_link3.stl" scale="0.001 0.001 0.001"/>
+      </geometry>
+      <material name="grey"/>
+    </visual>
+    <collision>
+      <origin xyz="0 0 0" rpy="0 0 0"/>
+      <geometry>
+        <mesh filename="file://$(find open_manipulator_description)/meshes/chain_link3.stl" scale="0.001 0.001 0.001"/>
       </geometry>
     </collision>
@@ -92,12 +92,12 @@
       <origin xyz="0 0 0" rpy="0 0 0"/>
       <geometry>
-        <mesh filename="package://open_manipulator_description/meshes/chain_link4.stl" scale="0.001 0.001 0.001"/>
-      </geometry>
-      <material name="grey"/>
-    </visual>
-    <collision>
-      <origin xyz="0 0 0" rpy="0 0 0"/>
-      <geometry>
-        <mesh filename="package://open_manipulator_description/meshes/chain_link4.stl" scale="0.001 0.001 0.001"/>
+        <mesh filename="file://$(find open_manipulator_description)/meshes/chain_link4.stl" scale="0.001 0.001 0.001"/>
+      </geometry>
+      <material name="grey"/>
+    </visual>
+    <collision>
+      <origin xyz="0 0 0" rpy="0 0 0"/>
+      <geometry>
+        <mesh filename="file://$(find open_manipulator_description)/meshes/chain_link4.stl" scale="0.001 0.001 0.001"/>
       </geometry>
     </collision>
@@ -121,12 +121,12 @@
       <origin xyz="0 0 0" rpy="0 0 0"/>
       <geometry>
-        <mesh filename="package://open_manipulator_description/meshes/chain_link5.stl" scale="0.001 0.001 0.001"/>
-      </geometry>
-      <material name="grey"/>
-    </visual>
-    <collision>
-      <origin xyz="0 0 0" rpy="0 0 0"/>
-      <geometry>
-        <mesh filename="package://open_manipulator_description/meshes/chain_link5.stl" scale="0.001 0.001 0.001"/>
+        <mesh filename="file://$(find open_manipulator_description)/meshes/chain_link5.stl" scale="0.001 0.001 0.001"/>
+      </geometry>
+      <material name="grey"/>
+    </visual>
+    <collision>
+      <origin xyz="0 0 0" rpy="0 0 0"/>
+      <geometry>
+        <mesh filename="file://$(find open_manipulator_description)/meshes/chain_link5.stl" scale="0.001 0.001 0.001"/>
       </geometry>
     </collision>
@@ -150,5 +150,5 @@
       <origin xyz="0.0 0.0 0" rpy="0 0 0"/>
       <geometry>
-        <mesh filename="package://open_manipulator_description/meshes/chain_link_grip_l.stl" scale="0.001 0.001 0.001"/>
+        <mesh filename="file://$(find open_manipulator_description)/meshes/chain_link_grip_l.stl" scale="0.001 0.001 0.001"/>
       </geometry>
       <material name="grey"/>
@@ -157,5 +157,5 @@
       <origin xyz="0.0 0.0 0" rpy="0 0 0"/>
       <geometry>
-        <mesh filename="package://open_manipulator_description/meshes/chain_link_grip_l.stl" scale="0.001 0.001 0.001"/>
+        <mesh filename="file://$(find open_manipulator_description)/meshes/chain_link_grip_l.stl" scale="0.001 0.001 0.001"/>
       </geometry>
     </collision>
@@ -180,5 +180,5 @@
       <origin xyz="0.0 -0.0 0" rpy="0 0 0"/>
       <geometry>
-        <mesh filename="package://open_manipulator_description/meshes/chain_link_grip_r.stl" scale="0.001 0.001 0.001"/>
+        <mesh filename="file://$(find open_manipulator_description)/meshes/chain_link_grip_r.stl" scale="0.001 0.001 0.001"/>
       </geometry>
       <material name="grey"/>
@@ -187,5 +187,5 @@
       <origin xyz="0.0 -0.0 0" rpy="0 0 0"/>
       <geometry>
-        <mesh filename="package://open_manipulator_description/meshes/chain_link_grip_r.stl" scale="0.001 0.001 0.001"/>
+        <mesh filename="file://$(find open_manipulator_description)/meshes/chain_link_grip_r.stl" scale="0.001 0.001 0.001"/>
       </geometry>
     </collision>

Commit message: Update robot description and simulation launch

File: src/open_manipulator_description/urdf/open_manipulator.xacro (robot description, xacro)
@@ -28,4 +28,5 @@
     <origin xyz="0.012 0.0 0.017" rpy="0 0 0"/>
     <axis xyz="0 0 1"/>
+    <dynamics damping="0.7" friction="1.0"/>
     <limit velocity="4.8" effort="1" lower="${-pi*0.9}" upper="${pi*0.9}" />
   </joint>
@@ -57,4 +58,5 @@
     <origin xyz="0.0 0.0 0.0595" rpy="0 0 0"/>
     <axis xyz="0 1 0"/>
+    <dynamics damping="0.7" friction="1.0"/>
     <limit velocity="4.8" effort="1" lower="${-pi*0.57}" upper="${pi*0.5}" />
   </joint>
@@ -86,4 +88,5 @@
     <origin xyz="0.024 0 0.128" rpy="0 0 0"/>
     <axis xyz="0 1 0"/>
+    <dynamics damping="0.7" friction="1.0"/>
     <limit velocity="4.8" effort="1" lower="${-pi*0.3}" upper="${pi*0.44}" />
   </joint>
@@ -115,4 +118,5 @@
     <origin xyz="0.124 0.0 0.0" rpy="0 0 0"/>
     <axis xyz="0 1 0"/>
+    <dynamics damping="0.7" friction="1.0"/>
     <limit velocity="4.8" effort="1" lower="${-pi*0.57}" upper="${pi*0.65}" />
   </joint>

File: src/open_manipulator_description/urdf/open_manipulator_robot.xacro (robot description, xacro)
@@ -4,25 +4,60 @@
   <xacro:include filename="$(find open_manipulator_description)/urdf/open_manipulator.xacro" />
   <link name="world"/>
-  <link name="base">
+  <link name="base_link">
       <visual>
         <geometry>
-          <cylinder length="0.6" radius="0.2"/>
+          <cylinder length="0.3" radius="0.3"/>
         </geometry>
       </visual>
       <collision>
         <geometry>
-          <cylinder length="0.6" radius="0.2"/>
+          <cylinder length="0.3" radius="0.3"/>
         </geometry>
       </collision>
    </link>
   <joint name="world_fixed" type="fixed">
-    <origin xyz="0 0 0.05" rpy="0 0 0"/>
+    <origin xyz="0 0 0.2" rpy="0 0 0"/>
     <parent link="world"/>
-    <child link="base"/>
+    <child link="base_link"/>
   </joint>
    <joint name="based_fixed" type="fixed">
-    <origin xyz="0 0 0.3" rpy="0 0 0"/>
-    <parent link="base"/>
+    <origin xyz="0 0 0.16" rpy="0 0 0"/>
+    <parent link="base_link"/>
     <child link="link1"/>
   </joint>
+  <gazebo>
+    <plugin name="gazebo_ros2_control" filename="libgazebo_ros2_control.so">
+      <parameters>$(find open_manipulator_control)/config/controllers.yaml</parameters>
+    </plugin>
+  </gazebo>
+  <xacro:macro name="manipulator_joint_command_by_position" params="name initial_value">
+    <joint name="${name}">
+        <command_interface name="position"/>
+        <state_interface name="position">
+          <param name="initial_value">${initial_value}</param>
+        </state_interface>
+        <state_interface name="velocity"/>
+    </joint>
+  </xacro:macro>
+  <ros2_control name="open_manipulator" type="system">
+    <hardware>
+      <plugin>gazebo_ros2_control/GazeboSystem</plugin>
+    </hardware>
+    <xacro:manipulator_joint_command_by_position name="joint1" initial_value="0"/>
+    <xacro:manipulator_joint_command_by_position name="joint2" initial_value="0"/>
+    <xacro:manipulator_joint_command_by_position name="joint3" initial_value="0"/>
+    <xacro:manipulator_joint_command_by_position name="joint4" initial_value="0"/>
+    <joint name="gripper">
+        <command_interface name="position"/>
+        <command_interface name="velocity"/>
+        <state_interface name="position"/>
+        <state_interface name="velocity"/>
+      </joint>
+    <joint name="gripper_sub">
+        <param name="mimic">gripper</param>
+        <param name="multiplier">-1</param>
+        <command_interface name="velocity"/>
+        <state_interface name="position"/>
+    </joint>
+  </ros2_control>
 </robot>

Commit message: Moved setup of ros2_control and remove end efector link

File: src/open_manipulator_description/urdf/open_manipulator.xacro (robot description, xacro)
@@ -202,24 +202,3 @@
     </inertial>
   </link>
-  <joint name="end_effector_joint" type="fixed">
-    <origin xyz="0.126 0.0 0.0" rpy="0 0 0"/>
-    <parent link="link5"/>
-    <child link="end_effector_link"/>
-  </joint>
-  <link name="end_effector_link">
-    <visual>
-      <origin xyz="0 0 0" rpy="0 0 0"/>
-      <geometry>
-        <box size="0.01 0.01 0.01" />
-      </geometry>
-      <material name="red"/>
-     </visual>
-    <inertial>
-      <origin xyz="0 0 0" />
-      <mass value="1.0e-03" />
-      <inertia ixx="1.0e-03" ixy="0.0" ixz="0.0"
-               iyy="1.0e-03" iyz="0.0"
-               izz="1.0e-03" />
-    </inertial>
-  </link>
 </robot>

File: src/open_manipulator_description/urdf/open_manipulator_robot.xacro (robot description, xacro)
@@ -3,4 +3,5 @@
   <xacro:include filename="$(find open_manipulator_description)/urdf/materials.xacro" />
   <xacro:include filename="$(find open_manipulator_description)/urdf/open_manipulator.xacro" />
+  <xacro:include filename="$(find open_manipulator_description)/urdf/ros2_control.xacro" />
   <link name="world"/>
   <link name="base_link">
@@ -26,38 +27,3 @@
     <child link="link1"/>
   </joint>
-  <gazebo>
-    <plugin name="gazebo_ros2_control" filename="libgazebo_ros2_control.so">
-      <parameters>$(find open_manipulator_control)/config/controllers.yaml</parameters>
-    </plugin>
-  </gazebo>
-  <xacro:macro name="manipulator_joint_command_by_position" params="name initial_value">
-    <joint name="${name}">
-        <command_interface name="position"/>
-        <state_interface name="position">
-          <param name="initial_value">${initial_value}</param>
-        </state_interface>
-        <state_interface name="velocity"/>
-    </joint>
-  </xacro:macro>
-  <ros2_control name="open_manipulator" type="system">
-    <hardware>
-      <plugin>gazebo_ros2_control/GazeboSystem</plugin>
-    </hardware>
-    <xacro:manipulator_joint_command_by_position name="joint1" initial_value="0"/>
-    <xacro:manipulator_joint_command_by_position name="joint2" initial_value="0"/>
-    <xacro:manipulator_joint_command_by_position name="joint3" initial_value="0"/>
-    <xacro:manipulator_joint_command_by_position name="joint4" initial_value="0"/>
-    <joint name="gripper">
-        <command_interface name="position"/>
-        <command_interface name="velocity"/>
-        <state_interface name="position"/>
-        <state_interface name="velocity"/>
-      </joint>
-    <joint name="gripper_sub">
-        <param name="mimic">gripper</param>
-        <param name="multiplier">-1</param>
-        <command_interface name="velocity"/>
-        <state_interface name="position"/>
-    </joint>
-  </ros2_control>
 </robot>

Commit message: Add basic configuation of moveit for open_manipulator

File: src/open_manipulator_description/urdf/open_manipulator.xacro (robot description, xacro)
@@ -202,3 +202,9 @@
     </inertial>
   </link>
+  <link name="end_efector_link" />
+  <joint name="end_efector" type="fixed">
+    <parent link="link5"/>
+    <child link="end_efector_link"/>
+    <origin xyz="0.1 0.0 0.0" rpy="0 0 0"/>
+  </joint>
 </robot>

File: src/open_manipulator_description/urdf/open_manipulator_robot.xacro (robot description, xacro)
@@ -31,3 +31,9 @@
     <child link="link1"/>
   </joint>
+  <link name="gripper_sub_mimic_link"/>
+  <joint name="gripper_sub_mimic" type="fixed">
+    <origin xyz="0 0 0" rpy="0 0 0"/>
+    <parent link="world"/>
+    <child link="gripper_sub_mimic_link"/>
+  </joint>
 </robot>

File: src/open_manipulator_description/urdf/ros2_control.xacro (robot description, xacro)
@@ -31,5 +31,5 @@
     <joint name="gripper_sub">
         <param name="mimic">gripper</param>
-        <param name="multiplier">-1</param>
+        <param name="multiplier">1</param>
         <command_interface name="velocity"/>
         <state_interface name="position"/>

Commit message: Use macro for manipulator links

File: src/open_manipulator_description/urdf/open_manipulator.xacro (robot description, xacro)
@@ -1,26 +1,32 @@
 <?xml version="1.0"?>
 <robot xmlns:xacro="http://ros.org/wiki/xacro">
-  <link name="link1">
-    <visual>
-      <origin xyz="0 0 0" rpy="0 0 0"/>
-      <geometry>
-        <mesh filename="file://$(find open_manipulator_description)/meshes/chain_link1.stl" scale="0.001 0.001 0.001"/>
-      </geometry>
-      <material name="grey"/>
-    </visual>
-    <collision>
-      <origin xyz="0 0 0" rpy="0 0 0"/>
-      <geometry>
-        <mesh filename="file://$(find open_manipulator_description)/meshes/chain_link1.stl" scale="0.001 0.001 0.001"/>
-      </geometry>
-    </collision>
+  <xacro:macro  name="arm_link" params="name *origin *inertial mesh_name">
+    <link name="${name}">
+      <xacro:insert_block name="inertial"/>
+      <visual>
+        <xacro:insert_block name="origin"/>
+        <geometry>
+          <mesh filename="file://$(find open_manipulator_description)/meshes/${mesh_name}" scale="0.001 0.001 0.001"/>
+        </geometry>
+        <material name="grey"/>
+      </visual>
+      <collision>
+        <xacro:insert_block name="origin"/>
+        <geometry>
+          <mesh filename="file://$(find open_manipulator_description)/meshes/${mesh_name}" scale="0.001 0.001 0.001"/>
+        </geometry>
+      </collision>
+    </link>
+  </xacro:macro>
+  <xacro:arm_link name="link1" mesh_name="chain_link1.stl">
+    <origin xyz="0 0 0" rpy="0 0 0"/>
     <inertial>
       <origin xyz="3.0876154e-04 0.0000000e+00 -1.2176461e-04" />
       <mass value="7.9119962e-02" />
       <inertia ixx="1.2505234e-05" ixy="0.0" ixz="-1.7855208e-07"
-               iyy="2.1898364e-05" iyz="0.0"
-               izz="1.9267361e-05" />
+              iyy="2.1898364e-05" iyz="0.0"
+              izz="1.9267361e-05" />
     </inertial>
-  </link>
+  </xacro:arm_link>
   <joint name="joint1" type="revolute">
     <parent link="link1"/>
@@ -31,18 +37,6 @@
     <limit velocity="4.8" effort="1" lower="${-pi*0.9}" upper="${pi*0.9}" />
   </joint>
-  <link name="link2">
-    <visual>
-      <origin xyz="0 0 0.019" rpy="0 0 0"/>
-      <geometry>
-        <mesh filename="file://$(find open_manipulator_description)/meshes/chain_link2.stl" scale="0.001 0.001 0.001"/>
-      </geometry>
-      <material name="grey"/>
-    </visual>
-    <collision>
-      <origin xyz="0 0 0.019" rpy="0 0 0"/>
-      <geometry>
-        <mesh filename="file://$(find open_manipulator_description)/meshes/chain_link2.stl" scale="0.001 0.001 0.001"/>
-      </geometry>
-    </collision>
+  <xacro:arm_link name="link2" mesh_name="chain_link2.stl">
+    <origin xyz="0 0 0.019" rpy="0 0 0"/>
     <inertial>
       <origin xyz="-3.0184870e-04 5.4043684e-04 ${0.018 + 2.9433464e-02}" />
@@ -52,5 +46,5 @@
                izz="1.8850320e-05" />
     </inertial>
-  </link>
+  </xacro:arm_link>
   <joint name="joint2" type="revolute">
     <parent link="link2"/>
@@ -61,18 +55,6 @@
     <limit velocity="4.8" effort="1" lower="${-pi*0.57}" upper="${pi*0.5}" />
   </joint>
-  <link name="link3">
-    <visual>
-      <origin xyz="0 0 0" rpy="0 0 0"/>
-      <geometry>
-        <mesh filename="file://$(find open_manipulator_description)/meshes/chain_link3.stl" scale="0.001 0.001 0.001"/>
-      </geometry>
-      <material name="grey"/>
-    </visual>
-    <collision>
-      <origin xyz="0 0 0" rpy="0 0 0"/>
-      <geometry>
-        <mesh filename="file://$(find open_manipulator_description)/meshes/chain_link3.stl" scale="0.001 0.001 0.001"/>
-      </geometry>
-    </collision>
+  <xacro:arm_link name="link3" mesh_name="chain_link3.stl">
+    <origin xyz="0 0 0" rpy="0 0 0"/>
     <inertial>
       <origin xyz="1.0308393e-02 3.7743363e-04 1.0170197e-01" />
@@ -82,5 +64,5 @@
                izz="6.0346498e-05" />
     </inertial>
-  </link>
+  </xacro:arm_link>
   <joint name="joint3" type="revolute">
     <parent link="link3"/>
@@ -91,18 +73,6 @@
     <limit velocity="4.8" effort="1" lower="${-pi*0.3}" upper="${pi*0.44}" />
   </joint>
-  <link name="link4">
-    <visual>
-      <origin xyz="0 0 0" rpy="0 0 0"/>
-      <geometry>
-        <mesh filename="file://$(find open_manipulator_description)/meshes/chain_link4.stl" scale="0.001 0.001 0.001"/>
-      </geometry>
-      <material name="grey"/>
-    </visual>
-    <collision>
-      <origin xyz="0 0 0" rpy="0 0 0"/>
-      <geometry>
-        <mesh filename="file://$(find open_manipulator_description)/meshes/chain_link4.stl" scale="0.001 0.001 0.001"/>
-      </geometry>
-    </collision>
+  <xacro:arm_link name="link4" mesh_name="chain_link4.stl">
+    <origin xyz="0 0 0" rpy="0 0 0"/>
     <inertial>
       <origin xyz="9.0909590e-02 3.8929816e-04 2.2413279e-04" />
@@ -112,5 +82,5 @@
                izz="2.5155057e-04" />
     </inertial>
-  </link>
+  </xacro:arm_link>
   <joint name="joint4" type="revolute">
     <parent link="link4"/>
@@ -121,18 +91,6 @@
     <limit velocity="4.8" effort="1" lower="${-pi*0.57}" upper="${pi*0.65}" />
   </joint>
-  <link name="link5">
-    <visual>
-      <origin xyz="0 0 0" rpy="0 0 0"/>
-      <geometry>
-        <mesh filename="file://$(find open_manipulator_description)/meshes/chain_link5.stl" scale="0.001 0.001 0.001"/>
-      </geometry>
-      <material name="grey"/>
-    </visual>
-    <collision>
-      <origin xyz="0 0 0" rpy="0 0 0"/>
-      <geometry>
-        <mesh filename="file://$(find open_manipulator_description)/meshes/chain_link5.stl" scale="0.001 0.001 0.001"/>
-      </geometry>
-    </collision>
+  <xacro:arm_link name="link5" mesh_name="chain_link5.stl">
+    <origin xyz="0 0 0" rpy="0 0 0"/>
     <inertial>
       <origin xyz="4.4206755e-02 3.6839985e-07 8.9142216e-03" />
@@ -142,5 +100,5 @@
                izz="9.3127351e-05" />
     </inertial>
-  </link>
+  </xacro:arm_link>
   <joint name="gripper" type="prismatic">
     <parent link="link5"/>
@@ -150,18 +108,6 @@
     <limit velocity="4.8" effort="1" lower="-0.010" upper="0.019" />
   </joint>
-  <link name="gripper_link">
-    <visual>
-      <origin xyz="0.0 0.0 0" rpy="0 0 0"/>
-      <geometry>
-        <mesh filename="file://$(find open_manipulator_description)/meshes/chain_link_grip_l.stl" scale="0.001 0.001 0.001"/>
-      </geometry>
-      <material name="grey"/>
-    </visual>
-    <collision>
-      <origin xyz="0.0 0.0 0" rpy="0 0 0"/>
-      <geometry>
-        <mesh filename="file://$(find open_manipulator_description)/meshes/chain_link_grip_l.stl" scale="0.001 0.001 0.001"/>
-      </geometry>
-    </collision>
+  <xacro:arm_link name="gripper_link" mesh_name="chain_link_grip_l.stl">
+    <origin xyz="0 0 0" rpy="0 0 0"/>
     <inertial>
       <origin xyz="0 0 0" />
@@ -171,5 +117,5 @@
                izz="1.0e-03" />
     </inertial>
-  </link>
+  </xacro:arm_link>
   <joint name="gripper_sub" type="prismatic">
     <parent link="link5"/>
@@ -180,18 +126,6 @@
     <mimic joint="gripper" multiplier="1"/>
   </joint>
-  <link name="gripper_link_sub">
-    <visual>
-      <origin xyz="0.0 -0.0 0" rpy="0 0 0"/>
-      <geometry>
-        <mesh filename="file://$(find open_manipulator_description)/meshes/chain_link_grip_r.stl" scale="0.001 0.001 0.001"/>
-      </geometry>
-      <material name="grey"/>
-    </visual>
-    <collision>
-      <origin xyz="0.0 -0.0 0" rpy="0 0 0"/>
-      <geometry>
-        <mesh filename="file://$(find open_manipulator_description)/meshes/chain_link_grip_r.stl" scale="0.001 0.001 0.001"/>
-      </geometry>
-    </collision>
+  <xacro:arm_link name="gripper_link_sub" mesh_name="chain_link_grip_r.stl">
+    <origin xyz="0 0 0" rpy="0 0 0"/>
     <inertial>
       <origin xyz="0 0 0" />
@@ -201,5 +135,5 @@
                izz="1.0e-03" />
     </inertial>
-  </link>
+  </xacro:arm_link>
   <link name="end_efector_link" />
   <joint name="end_efector" type="fixed">
