Commit message: Urdf of custom manipulator refactor

File: src/manipulator_6dof_description/urdf/manipulator_6dof_description.xacro (robot description, xacro)
@@ -3,7 +3,5 @@
   <xacro:include filename="$(find manipulator_6dof_description)/urdf/constants.xacro" />
   <xacro:include filename="$(find manipulator_6dof_description)/urdf/macros.xacro" />
-  <xacro:macro name="manipualtor_conectors" params="name r:=${pi/2} p:=0 y:=0">
-    <xacro:cylinder_link name="${name}" m="${manipualtor_conectors_mass}" hight="${manipualtor_conectors_hight}" radius="${manipualtor_conectors_radius}" xyz="0 0 0" rpy="${r} ${p} ${y}" />
-  </xacro:macro>
+  <xacro:include filename="$(find manipulator_6dof_description)/urdf/manipulator.xacro" />
   <link name="world"/>
   <xacro:cylinder_link
@@ -20,173 +18,9 @@
     <child link="base_link"/>
   </joint>
-  <xacro:cylinder_link
-    name="link1"
-    m="${link1_mass}"
-    hight="${link1_hight}"
-    radius="${link1_radius}"
-    xyz="0 0 0"
-    rpy="0 0 0" />
-  <joint name="based_fixed" type="fixed">
-    <origin xyz="0 0 ${offset_from_base_link_link1}" rpy="0 0 0"/>
-    <parent link="base_link"/>
-    <child link="link1"/>
-  </joint>
-  <xacro:cuboid_link
-    name="link2"
-    m="${link2_mass}"
-    x="${link2_depth}"
-    y="${link2_width}"
-    z="${link2_hight}"
-    xyz="0 0 0"
-    rpy="0 0 0" />
-  <joint name="joint1" type="revolute">
-    <parent link="link1"/>
-    <child link="link2"/>
-    <origin xyz="0 0 ${link2_hight/2 + joint_offest}" rpy="0 0 0"/>
-    <axis xyz="0 0 1"/>
-    <limit velocity="0" effort="0" lower="${-2.0*pi}" upper="${2.0*pi}" />
-  </joint>
-  <xacro:manipualtor_conectors name="link3" />
-  <joint name="joint2" type="revolute">
-    <origin
-      xyz="0 ${link2_width/2 + manipualtor_conectors_hight/2} ${link2_hight/2 - manipualtor_conectors_radius}"
-      rpy="0 0 0"/>
-    <parent link="link2"/>
-    <child link="link3"/>
-    <axis xyz="0 1 0"/>
-    <limit velocity="0" effort="0" lower="${-2.0*pi}" upper="${2.0*pi}" />
-  </joint>
-  <xacro:cuboid_link
-    name="link4"
-    m="${link4_mass}"
-    x="${link4_depth}"
-    y="${link4_width}"
-    z="${link4_hight}"
-    xyz="0 0 0"
-    rpy="0 0 0" />
-  <joint name="joint3" type="fixed">
-    <origin
-      xyz="${link4_depth/2 - manipualtor_conectors_radius} ${link4_width/2 + manipualtor_conectors_hight/2} 0"
-      rpy="0 0 0"/>
-    <parent link="link3"/>
-    <child link="link4"/>
-  </joint>
-  <xacro:manipualtor_conectors name="link5" />
-  <joint name="joint4" type="revolute">
-    <origin
-      xyz="${link4_depth/2 - manipualtor_conectors_radius} -${0.03 + manipualtor_conectors_hight/2} 0"
-      rpy="0 0 0" />
-    <parent link="link4"/>
-    <child link="link5"/>
-    <axis xyz="0 1 0"/>
-    <limit velocity="0" effort="0" lower="${-2.0*pi}" upper="${2.0*pi}" />
-  </joint>
-  <xacro:cuboid_link name="link6" m="${link6_mass}" x="${link6_depth}" y="${link6_width}" z="${link6_hight}" xyz="0 0 0" rpy="0 0 0" />
-  <joint name="joint5" type="fixed">
-    <origin
-      xyz="${link6_depth/2 - manipualtor_conectors_radius} -${link6_width/2 + manipualtor_conectors_hight/2} 0"
-      rpy="0 0 0"/>
-    <parent link="link5"/>
-    <child link="link6"/>
-  </joint>
-  <xacro:manipualtor_conectors name="link7" />
-  <joint name="joint6" type="revolute">
-    <origin
-      xyz="${link6_depth/2 - manipualtor_conectors_radius} ${link6_width/2 + manipualtor_conectors_hight/2} 0"
-      rpy="0 0 0" />
-    <parent link="link6" />
-    <child link="link7" />
-    <axis xyz="0 1 0" />
-    <limit velocity="0" effort="0" lower="${-2.0*pi}" upper="${2.0*pi}" />
-  </joint>
-  <xacro:cuboid_link
-    name="link8"
-    m="${link8_mass}"
-    x="${link8_depth}"
-    y="${link8_width}"
-    z="${link8_hight}"
-    xyz="0 0 0"
-    rpy="0 0 0" />
-  <joint name="joint7" type="fixed">
-    <origin
-      xyz="${manipualtor_conectors_hight} ${link8_width/2 + manipualtor_conectors_radius/2} 0"
-      rpy="0 0 0" />
-    <parent link="link7" />
-    <child link="link8" />
-  </joint>
-  <xacro:manipualtor_conectors name="link9" p="${pi/2}" r="0"/>
-  <joint name="joint8" type="revolute">
-    <origin xyz="${0.06+0.015} 0 0" rpy="0 0 0"/>
-    <parent link="link8"/>
-    <child link="link9"/>
-    <axis xyz="1 0 0"/>
-    <limit velocity="0" effort="0" lower="${-2.0*pi}" upper="${2.0*pi}" />
-  </joint>
-  <xacro:cuboid_link
-    name="link10"
-    m="${link10_mass}"
-    x="${link10_depth}"
-    y="${link10_width}"
-    z="${link10_hight}"
-    xyz="0 0 0"
-    rpy="${pi/2} 0 0" />
-  <joint name="joint9" type="fixed">
-    <origin
-      xyz="${link10_depth/2 + manipualtor_conectors_hight/2} 0 -${link10_width/2 - manipualtor_conectors_radius}"
-      rpy="0 0 0" />
-    <parent link="link9" />
-    <child link="link10" />
-  </joint>
-  <xacro:manipualtor_conectors name="link11" r="0"/>
-  <joint name="joint10" type="revolute">
-    <origin xyz="0 0 -${manipualtor_conectors_hight + link10_hight/2}" rpy="0 0 0"/>
-    <parent link="link10"/>
-    <child link="link11"/>
-    <axis xyz="0 0 1"/>
-    <limit velocity="0" effort="0" lower="${-2.0*pi}" upper="${2.0*pi}" />
-  </joint>
-  <xacro:cuboid_link
-    name="link12"
-    m="${link12_mass}"
-    x="${link12_depth}"
-    y="${link12_width}"
-    z="${link12_hight}"
-    xyz="0 0 0"
-    rpy="0 0 0" />
-  <joint name="joint11" type="fixed">
-    <origin xyz="0 0 -${link10_width/2 - manipualtor_conectors_radius}" rpy="0 0 0"/>
-    <parent link="link11"/>
-    <child link="link12"/>
-  </joint>
-  <xacro:cuboid_link
-    name="gripper_left"
-    m="${gripper_mass}"
-    x="${gripper_depth}"
-    y="${gripper_width}"
-    z="${gripper_hight}"
-    xyz="0 0 0"
-    rpy="0 0 0" />
-  <xacro:cuboid_link
-    name="gripper_right"
-    m="${gripper_mass}"
-    x="${gripper_depth}"
-    y="${gripper_width}"
-    z="${gripper_hight}"
-    xyz="0 0 0"
-    rpy="0 0 0" />
-  <joint name="joint12" type="prismatic">
-    <origin xyz="0 ${gripper_offset} -${gripper_hight/2 + link12_hight/2}" rpy="0 0 0"/>
-    <parent link="link12"/>
-    <child link="gripper_left"/>
-    <axis xyz="0 1 0"/>
-    <limit velocity="0" effort="0" lower="-0.025" upper="0.005" />
-  </joint>
-  <joint name="joint13" type="prismatic">
-    <origin xyz="0 -${gripper_offset} -${gripper_hight/2 + link12_hight/2}" rpy="0 0 0" />
-    <parent link="link12" />
-    <child link="gripper_right" />
-    <axis xyz="0 1 0" />
-    <limit velocity="0" effort="0" lower="-0.025" upper="0.005" />
-    <mimic joint="joint12" multiplier="-1"/>
+  <link name="gripper_right_mimic_link"/>
+  <joint name="gripper_right_mimic" type="fixed">
+    <origin xyz="0 0 0" rpy="0 0 0"/>
+    <parent link="world"/>
+    <child link="gripper_right_mimic_link"/>
   </joint>
 </robot>
