Commit message: Add ros2 control for custom manipulator

File: src/manipulator_6dof_description/urdf/macros.xacro (robot description, xacro)
@@ -26,6 +26,6 @@
   </xacro:macro>
   <xacro:macro name="cuboid_link" params="name m x y z xyz rpy">
-    <xacro:cuboid_inertia m="${m}" d="${x}" w="${y}" h="${z}" xyz="0 0 0" rpy="0 0 0"/>
     <link name="${name}">
+      <xacro:cuboid_inertia m="${m}" d="${x}" w="${y}" h="${z}" xyz="0 0 0" rpy="0 0 0"/>
       <visual>
         <origin xyz="${xyz}" rpy="${rpy}" />
@@ -36,4 +36,5 @@
       </visual>
       <collision>
+        <origin xyz="${xyz}" rpy="${rpy}" />
         <geometry>
           <box size="${x} ${y} ${z}" />
@@ -43,6 +44,6 @@
   </xacro:macro>
   <xacro:macro name="cylinder_link" params="name m hight radius xyz rpy color:=black">
-    <xacro:cylinder_inertia m="${m}" r="${radius}" h="${hight}" xyz="0 0 0" rpy="0 0 0"/>
     <link name="${name}">
+      <xacro:cylinder_inertia m="${m}" r="${radius}" h="${hight}" xyz="0 0 0" rpy="0 0 0"/>
       <visual>
         <origin xyz="${xyz}" rpy="${rpy}" />

File: src/manipulator_6dof_description/urdf/manipulator.xacro (robot description, xacro)
@@ -35,5 +35,5 @@
     <origin xyz="0 0 ${link2_hight/2 + joint_offest}" rpy="0 0 0"/>
     <axis xyz="0 0 1"/>
-    <limit velocity="0" effort="0" lower="${-2.0*pi}" upper="${2.0*pi}" />
+    <limit velocity="4.8" effort="1" lower="${-2.0*pi}" upper="${2.0*pi}" />
   </joint>
   <xacro:manipualtor_conectors name="link3" />
@@ -45,5 +45,5 @@
     <child link="link3"/>
     <axis xyz="0 1 0"/>
-    <limit velocity="0" effort="0" lower="${-2.0*pi}" upper="${2.0*pi}" />
+    <limit velocity="4.8" effort="1" lower="${-2.0*pi}" upper="${2.0*pi}" />
   </joint>
   <xacro:cuboid_link
@@ -70,5 +70,5 @@
     <child link="link5"/>
     <axis xyz="0 1 0"/>
-    <limit velocity="0" effort="0" lower="${-2.0*pi}" upper="${2.0*pi}" />
+    <limit velocity="4.8" effort="1" lower="${-2.0*pi}" upper="${2.0*pi}" />
   </joint>
   <xacro:cuboid_link name="link6" m="${link6_mass}" x="${link6_depth}" y="${link6_width}" z="${link6_hight}" xyz="0 0 0" rpy="0 0 0" />
@@ -88,5 +88,5 @@
     <child link="link7" />
     <axis xyz="0 1 0" />
-    <limit velocity="0" effort="0" lower="${-2.0*pi}" upper="${2.0*pi}" />
+    <limit velocity="4.8" effort="1" lower="${-2.0*pi}" upper="${2.0*pi}" />
   </joint>
   <xacro:cuboid_link
@@ -111,5 +111,5 @@
     <child link="link9"/>
     <axis xyz="1 0 0"/>
-    <limit velocity="0" effort="0" lower="${-2.0*pi}" upper="${2.0*pi}" />
+    <limit velocity="4.8" effort="1" lower="${-2.0*pi}" upper="${2.0*pi}" />
   </joint>
   <xacro:cuboid_link
@@ -134,5 +134,5 @@
     <child link="link11"/>
     <axis xyz="0 0 1"/>
-    <limit velocity="0" effort="0" lower="${-2.0*pi}" upper="${2.0*pi}" />
+    <limit velocity="4.8" effort="1" lower="${-2.0*pi}" upper="${2.0*pi}" />
   </joint>
   <xacro:cuboid_link
@@ -165,17 +165,17 @@
     xyz="0 0 0"
     rpy="0 0 0" />
-  <joint name="joint12" type="prismatic">
+  <joint name="gripper_left_joint" type="prismatic">
     <origin xyz="0 ${gripper_offset} -${gripper_hight/2 + link12_hight/2}" rpy="0 0 0"/>
     <parent link="link12"/>
     <child link="gripper_left"/>
     <axis xyz="0 1 0"/>
-    <limit velocity="0" effort="0" lower="-0.025" upper="0.005" />
+    <limit velocity="4.8" effort="1" lower="-0.025" upper="0.005" />
   </joint>
-  <joint name="joint13" type="prismatic">
+  <joint name="gripper_right_joint" type="prismatic">
     <origin xyz="0 -${gripper_offset} -${gripper_hight/2 + link12_hight/2}" rpy="0 0 0" />
     <parent link="link12" />
     <child link="gripper_right" />
     <axis xyz="0 1 0" />
-    <limit velocity="0" effort="0" lower="-0.025" upper="0.005" />
+    <limit velocity="4.8" effort="1" lower="-0.025" upper="0.005" />
     <mimic joint="joint12" multiplier="-1"/>
   </joint>

File: src/manipulator_6dof_description/urdf/manipulator_6dof_description.xacro (robot description, xacro)
@@ -1,7 +1,8 @@
 <?xml version="1.0"?>
-<robot name="open_manipulator" xmlns:xacro="http://ros.org/wiki/xacro">
+<robot name="manipulator_6dof" xmlns:xacro="http://ros.org/wiki/xacro">
   <xacro:include filename="$(find manipulator_6dof_description)/urdf/constants.xacro" />
   <xacro:include filename="$(find manipulator_6dof_description)/urdf/macros.xacro" />
   <xacro:include filename="$(find manipulator_6dof_description)/urdf/manipulator.xacro" />
+  <xacro:include filename="$(find manipulator_6dof_description)/urdf/ros2_control.xacro" />
   <link name="world"/>
   <xacro:cylinder_link
