Commit message: Add support of 3d sensor for 6dof manipualtor and fix spelling.

File: src/custom_6dof_manipulator/manipulator_6dof_description/urdf/constants.xacro (robot description, xacro)
@@ -2,43 +2,43 @@
 <robot xmlns:xacro="http://www.ros.org/wiki/xacro">
   <xacro:property name="joint_offest" value="0.01" />
-  <xacro:property name="base_link_hight" value="0.3" />
+  <xacro:property name="base_link_height" value="0.3" />
   <xacro:property name="base_link_radius" value="0.3" />
   <xacro:property name="base_link_mass" value="0.5" />
-  <xacro:property name="offset_from_ground_to_base_link" value="${base_link_hight/2 + 0.05}" />
-  <xacro:property name="offset_from_base_link_link1" value="${base_link_hight/2 + joint_offest}" />
-  <xacro:property name="manipualtor_conectors_hight" value="0.03" />
+  <xacro:property name="offset_from_ground_to_base_link" value="${base_link_height/2 + 0.05}" />
+  <xacro:property name="offset_from_base_link_link1" value="${base_link_height/2 + joint_offest}" />
+  <xacro:property name="manipualtor_conectors_height" value="0.03" />
   <xacro:property name="manipualtor_conectors_radius" value="0.03" />
   <xacro:property name="manipualtor_conectors_mass" value="0.3" />
   <xacro:property name="link1_mass" value="2" />
   <xacro:property name="link1_radius" value="0.1" />
-  <xacro:property name="link1_hight" value="0.1" />
+  <xacro:property name="link1_height" value="0.1" />
   <xacro:property name="link2_mass" value="1" />
   <xacro:property name="link2_depth" value="0.06" />
   <xacro:property name="link2_width" value="0.06" />
-  <xacro:property name="link2_hight" value="0.4" />
+  <xacro:property name="link2_height" value="0.4" />
   <xacro:property name="link4_mass" value="1" />
   <xacro:property name="link4_depth" value="0.4" />
   <xacro:property name="link4_width" value="0.06" />
-  <xacro:property name="link4_hight" value="0.06" />
+  <xacro:property name="link4_height" value="0.06" />
   <xacro:property name="link6_mass" value="0.5" />
   <xacro:property name="link6_depth" value="0.2" />
   <xacro:property name="link6_width" value="0.06" />
-  <xacro:property name="link6_hight" value="0.06" />
+  <xacro:property name="link6_height" value="0.06" />
   <xacro:property name="link8_mass" value="0.3" />
   <xacro:property name="link8_depth" value="0.12" />
   <xacro:property name="link8_width" value="0.06" />
-  <xacro:property name="link8_hight" value="0.06" />
+  <xacro:property name="link8_height" value="0.06" />
   <xacro:property name="link10_mass" value="0.2" />
   <xacro:property name="link10_depth" value="0.06" />
   <xacro:property name="link10_width" value="0.1" />
-  <xacro:property name="link10_hight" value="0.06" />
+  <xacro:property name="link10_height" value="0.06" />
   <xacro:property name="link12_mass" value="0.1" />
   <xacro:property name="link12_depth" value="0.01" />
   <xacro:property name="link12_width" value="0.08" />
-  <xacro:property name="link12_hight" value="0.01" />
+  <xacro:property name="link12_height" value="0.01" />
   <xacro:property name="gripper_mass" value="0.1" />
   <xacro:property name="gripper_depth" value="0.03" />
   <xacro:property name="gripper_width" value="0.01" />
-  <xacro:property name="gripper_hight" value="0.04" />
+  <xacro:property name="gripper_height" value="0.04" />
   <xacro:property name="gripper_offset" value="0.03" />
 </robot>

File: src/custom_6dof_manipulator/manipulator_6dof_description/urdf/macros.xacro (robot description, xacro)
@@ -43,7 +43,7 @@
     </link>
   </xacro:macro>
-  <xacro:macro name="cylinder_link" params="name m hight radius xyz rpy color:=black">
+  <xacro:macro name="cylinder_link" params="name m height radius xyz rpy color:=black">
     <link name="${name}">
-      <xacro:cylinder_inertia m="${m}" r="${radius}" h="${hight}" xyz="0 0 0" rpy="0 0 0"/>
+      <xacro:cylinder_inertia m="${m}" r="${radius}" h="${height}" xyz="0 0 0" rpy="0 0 0"/>
       <visual>
         <origin xyz="${xyz}" rpy="${rpy}" />

File: src/custom_6dof_manipulator/manipulator_6dof_description/urdf/manipulator.xacro (robot description, xacro)
@@ -5,5 +5,5 @@
       name="${name}"
       m="${manipualtor_conectors_mass}"
-      hight="${manipualtor_conectors_hight}"
+      height="${manipualtor_conectors_height}"
       radius="${manipualtor_conectors_radius}"
       xyz="0 0 0"
@@ -13,5 +13,5 @@
     name="link1"
     m="${link1_mass}"
-    hight="${link1_hight}"
+    height="${link1_height}"
     radius="${link1_radius}"
     xyz="0 0 0"
@@ -27,5 +27,5 @@
     x="${link2_depth}"
     y="${link2_width}"
-    z="${link2_hight}"
+    z="${link2_height}"
     xyz="0 0 0"
     rpy="0 0 0" />
@@ -33,5 +33,5 @@
     <parent link="link1"/>
     <child link="link2"/>
-    <origin xyz="0 0 ${link2_hight/2 + joint_offest}" rpy="0 0 0"/>
+    <origin xyz="0 0 ${link2_height/2 + joint_offest}" rpy="0 0 0"/>
     <axis xyz="0 0 1"/>
     <limit velocity="4.8" effort="1" lower="${-2.0*pi}" upper="${2.0*pi}" />
@@ -40,5 +40,5 @@
   <joint name="joint2" type="revolute">
     <origin
-      xyz="0 ${link2_width/2 + manipualtor_conectors_hight/2} ${link2_hight/2 - manipualtor_conectors_radius}"
+      xyz="0 ${link2_width/2 + manipualtor_conectors_height/2} ${link2_height/2 - manipualtor_conectors_radius}"
       rpy="0 0 0"/>
     <parent link="link2"/>
@@ -52,10 +52,10 @@
     x="${link4_depth}"
     y="${link4_width}"
-    z="${link4_hight}"
+    z="${link4_height}"
     xyz="0 0 0"
     rpy="0 0 0" />
   <joint name="joint3" type="fixed">
     <origin
-      xyz="${link4_depth/2 - manipualtor_conectors_radius} ${link4_width/2 + manipualtor_conectors_hight/2} 0"
+      xyz="${link4_depth/2 - manipualtor_conectors_radius} ${link4_width/2 + manipualtor_conectors_height/2} 0"
       rpy="0 0 0"/>
     <parent link="link3"/>
@@ -65,5 +65,5 @@
   <joint name="joint4" type="revolute">
     <origin
-      xyz="${link4_depth/2 - manipualtor_conectors_radius} -${manipualtor_conectors_hight + manipualtor_conectors_hight/2} 0"
+      xyz="${link4_depth/2 - manipualtor_conectors_radius} -${manipualtor_conectors_height + manipualtor_conectors_height/2} 0"
       rpy="0 0 0" />
     <parent link="link4"/>
@@ -72,8 +72,8 @@
     <limit velocity="4.8" effort="1" lower="${-2.0*pi}" upper="${2.0*pi}" />
   </joint>
-  <xacro:cuboid_link name="link6" m="${link6_mass}" x="${link6_depth}" y="${link6_width}" z="${link6_hight}" xyz="0 0 0" rpy="0 0 0" />
+  <xacro:cuboid_link name="link6" m="${link6_mass}" x="${link6_depth}" y="${link6_width}" z="${link6_height}" xyz="0 0 0" rpy="0 0 0" />
   <joint name="joint5" type="fixed">
     <origin
-      xyz="${link6_depth/2 - manipualtor_conectors_radius} -${link6_width/2 + manipualtor_conectors_hight/2} 0"
+      xyz="${link6_depth/2 - manipualtor_conectors_radius} -${link6_width/2 + manipualtor_conectors_height/2} 0"
       rpy="0 0 0"/>
     <parent link="link5"/>
@@ -83,5 +83,5 @@
   <joint name="joint6" type="revolute">
     <origin
-      xyz="${link6_depth/2 - manipualtor_conectors_radius} ${link6_width/2 + manipualtor_conectors_hight/2} 0"
+      xyz="${link6_depth/2 - manipualtor_conectors_radius} ${link6_width/2 + manipualtor_conectors_height/2} 0"
       rpy="0 0 0" />
     <parent link="link6" />
@@ -95,10 +95,10 @@
     x="${link8_depth}"
     y="${link8_width}"
-    z="${link8_hight}"
+    z="${link8_height}"
     xyz="0 0 0"
     rpy="0 0 0" />
   <joint name="joint7" type="fixed">
     <origin
-      xyz="${manipualtor_conectors_hight} ${link8_width/2 + manipualtor_conectors_radius/2} 0"
+      xyz="${manipualtor_conectors_height} ${link8_width/2 + manipualtor_conectors_radius/2} 0"
       rpy="0 0 0" />
     <parent link="link7" />
@@ -107,5 +107,5 @@
   <xacro:manipualtor_conectors name="link9" p="${pi/2}" r="0"/>
   <joint name="joint8" type="revolute">
-    <origin xyz="${link8_depth/2 + manipualtor_conectors_hight/2} 0 0" rpy="0 0 0"/>
+    <origin xyz="${link8_depth/2 + manipualtor_conectors_height/2} 0 0" rpy="0 0 0"/>
     <parent link="link8"/>
     <child link="link9"/>
@@ -118,10 +118,10 @@
     x="${link10_depth}"
     y="${link10_width}"
-    z="${link10_hight}"
+    z="${link10_height}"
     xyz="0 0 0"
     rpy="${pi/2} 0 0" />
   <joint name="joint9" type="fixed">
     <origin
-      xyz="${link10_depth/2 + manipualtor_conectors_hight/2} 0 -${link10_width/2 - manipualtor_conectors_radius}"
+      xyz="${link10_depth/2 + manipualtor_conectors_height/2} 0 -${link10_width/2 - manipualtor_conectors_radius}"
       rpy="0 0 0" />
     <parent link="link9" />
@@ -130,5 +130,5 @@
   <xacro:manipualtor_conectors name="link11" r="0"/>
   <joint name="joint10" type="revolute">
-    <origin xyz="0 0 -${manipualtor_conectors_hight/2 + link10_width/2}" rpy="0 0 0"/>
+    <origin xyz="0 0 -${manipualtor_conectors_height/2 + link10_width/2}" rpy="0 0 0"/>
     <parent link="link10"/>
     <child link="link11"/>
@@ -141,5 +141,5 @@
     x="${link12_depth}"
     y="${link12_width}"
-    z="${link12_hight}"
+    z="${link12_height}"
     xyz="0 0 0"
     rpy="0 0 0" />
@@ -154,5 +154,5 @@
     x="${gripper_depth}"
     y="${gripper_width}"
-    z="${gripper_hight}"
+    z="${gripper_height}"
     xyz="0 0 0"
     rpy="0 0 0" />
@@ -162,9 +162,9 @@
     x="${gripper_depth}"
     y="${gripper_width}"
-    z="${gripper_hight}"
+    z="${gripper_height}"
     xyz="0 0 0"
     rpy="0 0 0" />
   <joint name="gripper_left_joint" type="prismatic">
-    <origin xyz="0 ${gripper_offset} -${gripper_hight/2 + link12_hight/2}" rpy="0 0 0"/>
+    <origin xyz="0 ${gripper_offset} -${gripper_height/2 + link12_height/2}" rpy="0 0 0"/>
     <parent link="link12"/>
     <child link="gripper_left"/>
@@ -173,5 +173,5 @@
   </joint>
   <joint name="gripper_right_joint" type="prismatic">
-    <origin xyz="0 -${gripper_offset} -${gripper_hight/2 + link12_hight/2}" rpy="0 0 0" />
+    <origin xyz="0 -${gripper_offset} -${gripper_height/2 + link12_height/2}" rpy="0 0 0" />
     <parent link="link12" />
     <child link="gripper_right" />
@@ -184,5 +184,5 @@
     <parent link="link12"/>
     <child link="end_efector_link"/>
-    <origin xyz="0 0 -${gripper_hight/2 + link12_hight}" rpy="0 0 0"/>
+    <origin xyz="0 0 -${gripper_height/2 + link12_height}" rpy="0 0 0"/>
   </joint>
 </robot>

File: src/custom_6dof_manipulator/manipulator_6dof_description/urdf/manipulator_6dof_description.xacro (robot description, xacro)
@@ -5,9 +5,10 @@
   <xacro:include filename="$(find manipulator_6dof_description)/urdf/manipulator.xacro" />
   <xacro:include filename="$(find manipulator_6dof_description)/urdf/ros2_control.xacro" />
+  <xacro:include filename="$(find manipulator_6dof_description)/urdf/depth_camera.xacro" />
   <link name="world"/>
   <xacro:cylinder_link
     name="base_link"
     m="${base_link_mass}"
-    hight="${base_link_hight}"
+    height="${base_link_height}"
     radius="${base_link_radius}"
     xyz="0 0 0"

File: src/open_manipulator/open_manipulator_description/urdf/open_manipulator_robot.xacro (robot description, xacro)
@@ -4,18 +4,18 @@
   <xacro:include filename="$(find open_manipulator_description)/urdf/open_manipulator.xacro" />
   <xacro:include filename="$(find open_manipulator_description)/urdf/ros2_control.xacro" />
-  <xacro:property name="base_link_hight" value="0.3"/>
+  <xacro:property name="base_link_height" value="0.3"/>
   <xacro:property name="base_link_radius" value="0.3"/>
-  <xacro:property name="offset_from_ground_to_base_link" value="${base_link_hight/2 + 0.05}"/>
-  <xacro:property name="offset_from_base_link_link1" value="${base_link_hight/2 + 0.01}"/>
+  <xacro:property name="offset_from_ground_to_base_link" value="${base_link_height/2 + 0.05}"/>
+  <xacro:property name="offset_from_base_link_link1" value="${base_link_height/2 + 0.01}"/>
   <link name="world"/>
   <link name="base_link">
       <visual>
         <geometry>
-          <cylinder length="${base_link_hight}" radius="${base_link_radius}"/>
+          <cylinder length="${base_link_height}" radius="${base_link_radius}"/>
         </geometry>
       </visual>
       <collision>
         <geometry>
-          <cylinder length="${base_link_hight}" radius="${base_link_radius}"/>
+          <cylinder length="${base_link_height}" radius="${base_link_radius}"/>
         </geometry>
       </collision>
