Commit message: Add moveit for custom robot

File: src/custom_6dof_manipulator/manipulator_6dof_description/urdf/manipulator.xacro (robot description, xacro)
@@ -178,5 +178,5 @@
     <axis xyz="0 1 0" />
     <limit velocity="4.8" effort="1" lower="-0.025" upper="0.005" />
-    <mimic joint="joint12" multiplier="-1"/>
+    <mimic joint="gripper_left_joint" multiplier="-1"/>
   </joint>
   <link name="end_efector_link" />
@@ -184,5 +184,5 @@
     <parent link="link12"/>
     <child link="end_efector_link"/>
-    <origin xyz="0 0 -${gripper_hight/2 + link12_hight/2}" rpy="0 0 0"/>
+    <origin xyz="0 0 -${gripper_hight/2 + link12_hight}" rpy="0 0 0"/>
   </joint>
 </robot>

File: src/custom_6dof_manipulator/manipulator_6dof_description/urdf/manipulator_6dof_description.xacro (robot description, xacro)
@@ -20,5 +20,5 @@
   </joint>
   <link name="gripper_right_mimic_link"/>
-  <joint name="gripper_right_mimic" type="fixed">
+  <joint name="gripper_right_joint_mimic" type="fixed">
     <origin xyz="0 0 0" rpy="0 0 0"/>
     <parent link="world"/>

Commit message: Update custom 6DoF manipulator remove useless dummy link, and new state and cmd interfaces,add ode parameters for gripper.

File: src/custom_6dof_manipulator/manipulator_6dof_description/urdf/manipulator.xacro (robot description, xacro)
@@ -178,7 +178,17 @@
     <child link="gripper_right" />
     <axis xyz="0 1 0" />
-    <limit velocity="4.8" effort="1" lower="-0.025" upper="0.005" />
+    <limit velocity="4.8" effort="1" lower="0.025" upper="-0.005" />
     <mimic joint="gripper_left_joint" multiplier="-1"/>
   </joint>
+  <gazebo reference="gripper_left">
+    <mu1>10</mu1>
+    <mu2>10</mu2>
+    <minDepth>0.02</minDepth>
+  </gazebo>
+  <gazebo reference="gripper_right">
+    <mu1>10</mu1>
+    <mu2>10</mu2>
+    <minDepth>0.02</minDepth>
+  </gazebo>
   <link name="end_efector_link" />
   <joint name="end_efector" type="fixed">

File: src/custom_6dof_manipulator/manipulator_6dof_description/urdf/manipulator_6dof_description.xacro (robot description, xacro)
@@ -20,9 +20,3 @@
     <child link="base_link"/>
   </joint>
-  <link name="gripper_right_mimic_link"/>
-  <joint name="gripper_right_joint_mimic" type="fixed">
-    <origin xyz="0 0 0" rpy="0 0 0"/>
-    <parent link="world"/>
-    <child link="gripper_right_mimic_link"/>
-  </joint>
 </robot>

File: src/custom_6dof_manipulator/manipulator_6dof_description/urdf/ros2_control.xacro (robot description, xacro)
@@ -34,6 +34,8 @@
         <param name="mimic">gripper_left_joint</param>
         <param name="multiplier">-1</param>
+        <command_interface name="position"/>
         <command_interface name="velocity"/>
         <state_interface name="position"/>
+        <state_interface name="velocity"/>
     </joint>
   </ros2_control>
