Commit message: Migrate robots urdf to gazebo ignition

File: src/custom_6dof_manipulator/manipulator_6dof_description/urdf/depth_camera.xacro (robot description, xacro)
@@ -43,9 +43,4 @@
     </clip>
     </camera>
-      <plugin name="camera_controller" filename="libgazebo_ros_camera.so">
-        <frame_name>camera_link_optical</frame_name>
-        <min_depth>0.2</min_depth>
-        <max_depth>10.0</max_depth>
-      </plugin>
     </sensor>
   </gazebo>

File: src/custom_6dof_manipulator/manipulator_6dof_description/urdf/manipulator.xacro (robot description, xacro)
@@ -35,5 +35,5 @@
     <origin xyz="0 0 ${link2_height/2 + joint_offest}" rpy="0 0 0"/>
     <axis xyz="0 0 1"/>
-    <limit velocity="4.8" effort="1" lower="${-2.0*pi}" upper="${2.0*pi}" />
+    <limit velocity="4.8" effort="20" lower="${-2.0*pi}" upper="${2.0*pi}" />
   </joint>
   <xacro:manipualtor_conectors name="link3" />
@@ -45,5 +45,6 @@
     <child link="link3"/>
     <axis xyz="0 1 0"/>
-    <limit velocity="4.8" effort="1" lower="${-2.0*pi}" upper="${2.0*pi}" />
+    <dynamics damping="1.2" friction="1.5"/>
+    <limit velocity="4.8" effort="20" lower="${-2.0*pi}" upper="${2.0*pi}" />
   </joint>
   <xacro:cuboid_link
@@ -70,5 +71,5 @@
     <child link="link5"/>
     <axis xyz="0 1 0"/>
-    <limit velocity="4.8" effort="1" lower="${-2.0*pi}" upper="${2.0*pi}" />
+    <limit velocity="4.8" effort="20" lower="${-2.0*pi}" upper="${2.0*pi}" />
   </joint>
   <xacro:cuboid_link name="link6" m="${link6_mass}" x="${link6_depth}" y="${link6_width}" z="${link6_height}" xyz="0 0 0" rpy="0 0 0" />
@@ -88,7 +89,7 @@
     <child link="link7" />
     <axis xyz="0 1 0" />
-    <limit velocity="4.8" effort="1" lower="${-2.0*pi}" upper="${2.0*pi}" />
+    <limit velocity="4.8" effort="20" lower="${-2.0*pi}" upper="${2.0*pi}" />
   </joint>
-  <xacro:cuboid_link
+   <xacro:cuboid_link
     name="link8"
     m="${link8_mass}"
@@ -111,5 +112,5 @@
     <child link="link9"/>
     <axis xyz="1 0 0"/>
-    <limit velocity="4.8" effort="1" lower="${-2.0*pi}" upper="${2.0*pi}" />
+    <limit velocity="4.8" effort="20" lower="${-2.0*pi}" upper="${2.0*pi}" />
   </joint>
   <xacro:cuboid_link
@@ -134,5 +135,5 @@
     <child link="link11"/>
     <axis xyz="0 0 1"/>
-    <limit velocity="4.8" effort="1" lower="${-2.0*pi}" upper="${2.0*pi}" />
+    <limit velocity="4.8" effort="20" lower="${-2.0*pi}" upper="${2.0*pi}" />
   </joint>
   <xacro:cuboid_link

File: src/custom_6dof_manipulator/manipulator_6dof_description/urdf/ros2_control.xacro (robot description, xacro)
@@ -2,5 +2,5 @@
 <robot xmlns:xacro="http://ros.org/wiki/xacro">
   <gazebo>
-    <plugin name="gazebo_ros2_control" filename="libgazebo_ros2_control.so">
+    <plugin name="ign_ros2_control::IgnitionROS2ControlPlugin" filename="libign_ros2_control-system.so" >
       <parameters>$(find manipulator_6dof_control)/config/controllers.yaml</parameters>
     </plugin>
@@ -17,5 +17,5 @@
   <ros2_control name="6dof_manipulator" type="system">
     <hardware>
-      <plugin>gazebo_ros2_control/GazeboSystem</plugin>
+      <plugin>ign_ros2_control/IgnitionSystem</plugin>
     </hardware>
     <xacro:manipulator_joint_command_by_position name="joint1" initial_value="0"/>
@@ -24,5 +24,5 @@
     <xacro:manipulator_joint_command_by_position name="joint6" initial_value="0"/>
     <xacro:manipulator_joint_command_by_position name="joint8" initial_value="0"/>
-    <xacro:manipulator_joint_command_by_position name="joint10" initial_value="0"/>
+   <xacro:manipulator_joint_command_by_position name="joint10" initial_value="0"/>
     <joint name="gripper_left_joint">
         <command_interface name="position"/>

File: src/open_manipulator/open_manipulator_description/urdf/ros2_control.xacro (robot description, xacro)
@@ -2,5 +2,5 @@
 <robot xmlns:xacro="http://ros.org/wiki/xacro">
   <gazebo>
-    <plugin name="gazebo_ros2_control" filename="libgazebo_ros2_control.so">
+    <plugin name="ign_ros2_control::IgnitionROS2ControlPlugin" filename="libign_ros2_control-system.so" >
       <parameters>$(find open_manipulator_control)/config/controllers.yaml</parameters>
     </plugin>
@@ -17,5 +17,5 @@
   <ros2_control name="open_manipulator" type="system">
     <hardware>
-      <plugin>gazebo_ros2_control/GazeboSystem</plugin>
+      <plugin>ign_ros2_control/IgnitionSystem</plugin>
     </hardware>
     <xacro:manipulator_joint_command_by_position name="joint1" initial_value="0"/>

Commit message: Add depthe camera

File: src/custom_6dof_manipulator/manipulator_6dof_description/urdf/depth_camera.xacro (robot description, xacro)
@@ -14,4 +14,7 @@
         <box size="${camera_depth} ${camera_width} ${camera_height}"/>
       </geometry>
+        <material name="blue">
+        <color rgba="0 0 0.8 1"/>
+      </material>
     </visual>
     <collision>
@@ -20,27 +23,50 @@
       </geometry>
     </collision>
+    <inertial>
+      <origin xyz="0 0 0" rpy="0 0 0"/>
+      <mass value="0.01"/>
+      <inertia ixx="0.00001" ixy="0.0" ixz="0.0" iyy="0.00001" iyz="0.0" izz="0.00001"/>
+    </inertial>
   </link>
   <joint name="camera_optical_joint" type="fixed">
     <parent link="camera_link"/>
     <child link="camera_link_optical"/>
-    <origin xyz="0 0 0" rpy="${-pi/2} 0 ${-pi/2}"/>
+    <origin xyz="0 0 0" rpy="0 0 0"/>
   </joint>
   <link name="camera_link_optical"></link>
   <gazebo reference="camera_link">
-    <sensor name="camera" type="depth">
-    <visualize>true</visualize>
-    <update_rate>10</update_rate>
-    <camera>
-    <horizontal_fov>1.089</horizontal_fov>
-    <image>
-      <format>B8G8R8</format>
-      <width>640</width>
-      <height>480</height>
-    </image>
-    <clip>
-      <near>0.05</near>
-      <far>8.0</far>
-    </clip>
-    </camera>
+    <sensor name="camera" type="rgbd_camera">
+      <visualize>true</visualize>
+      <always_on>true</always_on>
+      <update_rate>30</update_rate>
+      <topic>camera</topic>
+      <enable_metrics>false</enable_metrics>
+      <camera>
+        <horizontal_fov>1.089</horizontal_fov>
+        <image>
+          <width>640</width>
+          <height>480</height>
+          <format>R8G8B8</format>
+        </image>
+        <clip>
+          <near>0.05</near>
+          <far>8.0</far>
+        </clip>
+        <lens>
+          <intrinsics>
+            <fx>554.25469</fx>
+            <fy>554.25469</fy>
+            <cx>320.5</cx>
+            <cy>240.5</cy>
+            <s>0</s>
+          </intrinsics>
+        </lens>
+        <noise>
+          <type>gaussian</type>
+          <mean>0.0</mean>
+          <stddev>0.007</stddev>
+        </noise>
+        <optical_frame_id>camera_link_optical</optical_frame_id>
+      </camera>
     </sensor>
   </gazebo>

File: src/open_manipulator/open_manipulator_description/urdf/open_manipulator_robot.xacro (robot description, xacro)
@@ -4,4 +4,5 @@
   <xacro:include filename="$(find open_manipulator_description)/urdf/open_manipulator.xacro" />
   <xacro:include filename="$(find open_manipulator_description)/urdf/ros2_control.xacro" />
+  <xacro:include filename="$(find open_manipulator_description)/urdf/depth_camera.xacro" />
   <xacro:property name="base_link_height" value="0.3"/>
   <xacro:property name="base_link_radius" value="0.3"/>
