Commit message: Increase effort limit for open_manipulators joints

File: src/open_manipulator/open_manipulator_description/urdf/open_manipulator.xacro (robot description, xacro)
@@ -35,5 +35,5 @@
     <axis xyz="0 0 1"/>
     <dynamics damping="0.7" friction="1.0"/>
-    <limit velocity="4.8" effort="1" lower="${-pi*0.9}" upper="${pi*0.9}" />
+    <limit velocity="4.8" effort="5" lower="${-pi*0.9}" upper="${pi*0.9}" />
   </joint>
   <xacro:arm_link name="link2" mesh_name="chain_link2.stl">
@@ -53,5 +53,5 @@
     <axis xyz="0 1 0"/>
     <dynamics damping="0.7" friction="1.0"/>
-    <limit velocity="4.8" effort="1" lower="${-pi*0.57}" upper="${pi*0.5}" />
+    <limit velocity="4.8" effort="5" lower="${-pi*0.57}" upper="${pi*0.5}" />
   </joint>
   <xacro:arm_link name="link3" mesh_name="chain_link3.stl">
@@ -71,5 +71,5 @@
     <axis xyz="0 1 0"/>
     <dynamics damping="0.7" friction="1.0"/>
-    <limit velocity="4.8" effort="1" lower="${-pi*0.3}" upper="${pi*0.44}" />
+    <limit velocity="4.8" effort="5" lower="${-pi*0.3}" upper="${pi*0.44}" />
   </joint>
   <xacro:arm_link name="link4" mesh_name="chain_link4.stl">
@@ -89,5 +89,5 @@
     <axis xyz="0 1 0"/>
     <dynamics damping="0.7" friction="1.0"/>
-    <limit velocity="4.8" effort="1" lower="${-pi*0.57}" upper="${pi*0.65}" />
+    <limit velocity="4.8" effort="5" lower="${-pi*0.57}" upper="${pi*0.65}" />
   </joint>
   <xacro:arm_link name="link5" mesh_name="chain_link5.stl">
@@ -106,5 +106,5 @@
     <origin xyz="0.0817 0.021 0.0" rpy="0 0 0"/>
     <axis xyz="0 1 0"/>
-    <limit velocity="4.8" effort="1" lower="-0.010" upper="0.019" />
+    <limit velocity="4.8" effort="5" lower="-0.010" upper="0.019" />
   </joint>
   <xacro:arm_link name="gripper_link" mesh_name="chain_link_grip_l.stl">
@@ -123,5 +123,5 @@
     <origin xyz="0.0817 -0.021 0" rpy="0 0 0"/>
     <axis xyz="0 -1 0"/>
-    <limit velocity="4.8" effort="1" lower="-0.010" upper="0.019" />
+    <limit velocity="4.8" effort="5" lower="-0.010" upper="0.019" />
     <mimic joint="gripper" multiplier="1"/>
   </joint>
