Commit message: Remove useless dummy link from open manipulator and new command and state interfaces for gripper

File: src/open_manipulator/open_manipulator_description/urdf/open_manipulator_robot.xacro (robot description, xacro)
@@ -31,9 +31,3 @@
     <child link="link1"/>
   </joint>
-  <link name="gripper_sub_mimic_link"/>
-  <joint name="gripper_sub_mimic" type="fixed">
-    <origin xyz="0 0 0" rpy="0 0 0"/>
-    <parent link="world"/>
-    <child link="gripper_sub_mimic_link"/>
-  </joint>
 </robot>

File: src/open_manipulator/open_manipulator_description/urdf/ros2_control.xacro (robot description, xacro)
@@ -32,6 +32,8 @@
         <param name="mimic">gripper</param>
         <param name="multiplier">1</param>
+        <command_interface name="position"/>
         <command_interface name="velocity"/>
         <state_interface name="position"/>
+        <state_interface name="velocity"/>
     </joint>
   </ros2_control>
